File: controlSemaforicoMEga.kicad_pcb (KiCad board)
At the start: 2 copper layers, 114 x 105.1 mm, 2 parts, among them J2 Conn_01x44_Socket

Commit message: V1
Parts:
- added J1: MicroSD, Connector_PinHeader_2.54mm:PinHeader_1x06_P2.54mm_Vertical, F.Cu at (126.0, 61.0)
- added J3: GPS, Connector_PinHeader_2.54mm:PinHeader_1x04_P2.54mm_Vertical, F.Cu at (139.8, 58.7)
- added J4: RTC, Connector_PinHeader_2.54mm:PinHeader_1x04_P2.54mm_Vertical, B.Cu at (157.3, 59.3)
- added J5: LCD, Connector_PinHeader_2.54mm:PinHeader_1x04_P2.54mm_Vertical, F.Cu at (186.8, 45.6)
Connections:
- A1 pad 5V1: unconnected-(A1-5V-Pad5V1) -> VCC
- A1 pad 5V4: unconnected-(A1-5V-Pad5V4) -> VCC
- A1 pad D18: unconnected-(A1-D18/TX1-PadD18) -> Net-(A1-D18/TX1)
- A1 pad D19: unconnected-(A1-D19/RX1-PadD19) -> Net-(A1-D19/RX1)
- A1 pad D50: unconnected-(A1-D50_MISO-PadD50) -> Net-(A1-D50_MISO)
- A1 pad D51: unconnected-(A1-D51_MOSI-PadD51) -> Net-(A1-D51_MOSI)
- A1 pad D52: unconnected-(A1-D52_SCK-PadD52) -> Net-(A1-D52_SCK)
- A1 pad D53: unconnected-(A1-D53_CS-PadD53) -> Net-(A1-D53_CS)
- A1 pad SCL: unconnected-(A1-PadSCL) -> Net-(J4-Pin_4)
- A1 pad SDA: unconnected-(A1-PadSDA) -> Net-(J4-Pin_3)
Routing:
- net Net-(A1-D18/TX1): track 0.00 -> 140.7 mm, vias 0 -> 1
- net Net-(A1-D19/RX1): track 0.00 -> 131.6 mm, vias 0 -> 1
- net Net-(J4-Pin_3): track 0.00 -> 103.9 mm
- net Net-(J4-Pin_4): track 0.00 -> 102.5 mm
- net VCC: track 26.4 -> 128.5 mm
- net Net-(A1-D51_MOSI): track 0.00 -> 86.2 mm
- net Net-(A1-D53_CS): track 0.00 -> 68.6 mm
- net Net-(A1-D52_SCK): track 0.00 -> 61.2 mm
- net Net-(A1-D50_MISO): track 0.00 -> 57.0 mm

Commit message: update
Parts:
- added J6: I2C, Connector_PinHeader_2.54mm:PinHeader_1x04_P2.54mm_Vertical, F.Cu at (132.8, 52.3)
- moved J5 7.09 mm to (193.6, 43.6)
Routing:
- net Net-(J4-Pin_4): track 102.5 -> 137.8 mm, vias 0 -> 1
- net Net-(J4-Pin_3): track 103.9 -> 137.9 mm
- net VCC: track 128.5 -> 143.2 mm
