File: controlSemaforicoMEga.kicad_sch (KiCad schematic)
At the start: 2 parts, among them J2 Conn_01x44_Socket

Commit message: V1
Parts:
- added J1: MicroSD, Connector_PinHeader_2.54mm:PinHeader_1x06_P2.54mm_Vertical, symbol Connector:Conn_01x06_Pin
- added J3: GPS, Connector_PinHeader_2.54mm:PinHeader_1x04_P2.54mm_Vertical, symbol Connector:Conn_01x04_Pin
- added J4: RTC, Connector_PinHeader_2.54mm:PinHeader_1x04_P2.54mm_Vertical, symbol Connector:Conn_01x04_Pin
- added J5: LCD, Connector_PinHeader_2.54mm:PinHeader_1x04_P2.54mm_Vertical, symbol Connector:Conn_01x04_Pin
Connections:
- net GND: now also J1.1 (Pin_1), J3.1 (Pin_1), J4.1 (Pin_1), J5.1 (Pin_1)
- net VCC: now also A1.5V1 (5V), A1.5V4 (5V), J1.2 (Pin_2), J3.4 (Pin_4), J4.2 (Pin_2), J5.2 (Pin_2)
- net at A1.D18 (D18/TX1): now also J3.3 (Pin_3)
- net at A1.D19 (D19/RX1): now also J3.2 (Pin_2)
- net at A1.D50 (D50_MISO): now also J1.3 (Pin_3)
- net at A1.D51 (D51_MOSI): now also J1.4 (Pin_4)
- net at A1.D52 (D52_SCK): now also J1.5 (Pin_5)
- net at A1.D53 (D53_CS): now also J1.6 (Pin_6)
- net at A1.SCL: now also J4.4 (Pin_4), J5.3 (Pin_3)
- net at A1.SDA: now also J4.3 (Pin_3), J5.4 (Pin_4)

Commit message: update
Parts:
- added J6: I2C, Connector_PinHeader_2.54mm:PinHeader_1x04_P2.54mm_Vertical, symbol Connector:Conn_01x04_Pin
Connections:
- net GND: now also J6.1 (Pin_1)
- net VCC: now also J6.2 (Pin_2)
- net at A1.SCL, J4.4 (Pin_4), J5.3 (Pin_3): now also J6.3 (Pin_3)
- net at A1.SDA, J4.3 (Pin_3), J5.4 (Pin_4): now also J6.4 (Pin_4)

Commit message: add title
Other:
- title: (none) -> Tarjeta de Control (Mega)
Changed lines of the file:
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@@
 	(generator_version "8.0")
 	(paper "A4")
+	(title_block
+		(title "Tarjeta de Control (Mega)")
+	)
 	(junction
 		(at 80.01 101.6)
